File: layout/control.sch (EAGLE design)
At the start: 9 parts, among them IC1 ATMEGA328", U1 RESONATOR"

Commit message: wip
Parts:
- added C1, C2: 47uF, RBBB:ELECTROLYTIC_CAP2.54MM
- added D1: 1N4004, diode:1N4004
- added IC2: (no value), RBBB:REGULATOR
- added J1: POWER_JACK", RBBB:POWER_JACK"
- added JP2: (no value), RBBB:1X04_HEADER"
- added SV1: (no value), con-lstb:MA08-1
- added U$1: 1X02_HEADER, RBBB:1X02_HEADER
- C3: device RBBB:ELECTROLYTIC_CAP2.54MM -> RBBB:UNPOLARIZED_CAP"
Connections:
- new net N$6: C2.+, D1.C, IC2.IN, J1.PWR, U$1.1
- net +5V: now also C1.+, C3.1, IC2.OUT, JP2.3; no longer C3.+
- net D10: now also SV1.6
- net D11: now also SV1.7
- net D12: now also SV1.8
- net D2: now also JP2.4
- net D5: now also SV1.1
- net D6: now also SV1.2
- net D7: now also SV1.3
- net D8: now also SV1.4
- net D9: now also SV1.5
- net GND: now also C1.-, C2.-, C3.2, D1.A, IC2.GND, JP2.2, U$1.2; no longer C3.-
