File: layout/newcontrol.sch (EAGLE design)
At the start: 7 parts, among them IC1 ATMEGA328", U1 RESONATOR"

Commit message: Finish controler layout!
Parts:
- added C1, C4: 0.1uF, RBBB:UNPOLARIZED_CAP"
- added C2: 47uF, RBBB:ELECTROLYTIC_CAP2.54MM
- added D1: 1N4004, diode:1N4004
- added IC2: (no value), RBBB:REGULATOR
- added J1: POWER_JACK", RBBB:POWER_JACK"
- added JP1: (no value), RBBB:1X06_HEADER"
- added U$1: 1X02_HEADER, RBBB:1X02_HEADER
- C3: value 0.1uF -> 47uF
Connections:
- new net A0: IC1.(PCI8/ADC0)PC0
- new net A1: IC1.(PCI9/ADC1)PC1
- new net A2: IC1.(PCI10/ADC2)PC2
- new net A3: IC1.(PCI11/ADC3)PC3
- new net A4: IC1.(PCI12/ADC4/SDA)PC4
- new net A5: IC1.(PCI13/ADC5/SCL)PC5
- new net AREF: IC1.AREF
- new net D0/RX: IC1.(PCI16/RXD)PD0, JP1.3
- new net D1/TX: IC1.(PCI17/TXD)PD1, JP1.2
- new net D10: IC1.(PCI2/SS/OC1B)PB2
- new net D11: IC1.(PCI3/MOSI/OC2A)PB3
- new net D12: IC1.(PCI4/MISO)PB4
- new net D13: IC1.(PCI5/SCK)PB5
- new net D2: IC1.(PCI18/INT0)PD2
- new net D3: IC1.(PCI19/INT1/OC2B)PD3
- new net D4: IC1.(PCI20/XCK/T0)PD4
- new net D5: IC1.(PCI21/T1/OC0B)PD5
- new net D6: IC1.(PCI22/AIN0OC0A)PD6
- new net D7: IC1.(PCI23/AIN1)PD7
- new net D8: IC1.(PCI0/ICP/CLKO)PB0
- new net D9: IC1.(PCI1/OC1A/OC1S)PB1
- new net EXT_RESET: C4.2, JP1.1
- new net N$5: C2.+, D1.C, IC2.IN, J1.PWR, U$1.1
- net +5V: now also C1.1, IC2.OUT, JP1.4
- net GND: now also C1.2, C2.-, D1.A, IC2.GND, J1.GND, J1.GNDBREAK, JP1.6, U$1.2
- net N$4: now also C4.1
Other:
- moved on the sheet: C3, IC1, U1
