File: layout/prototype.brd (EAGLE design)
At the start: 100 x 80 mm, 17 parts, among them IC1 ATMEGA328", J1 POWER_JACK", U1 RESONATOR"

Commit message: Finish controler layout!
Parts:
- removed JP2: (no value), RBBB:1X04_HEADER
- removed SV1: (no value), con-lstb:MA08-1
- added KEYPAD: 1X09_HEADER", RBBB:1X09_HEADER
- added RF: (no value), RBBB:1X04_HEADER
- C1: value 47uF -> 0.1uF; device RBBB:ELECTROLYTIC_CAP -> RBBB:UNPOLARIZED_CAP
- C3: value 0.1uF -> 47uF; device RBBB:UNPOLARIZED_CAP -> RBBB:ELECTROLYTIC_CAP
- moved JP1 53.6 mm to (3.81, 25.4), turned to 270 degrees
- moved R1 44.7 mm to (8.89, 17.8), turned to 90 degrees
- moved S1 35.2 mm to (15.2, 18.4), turned to 270 degrees
- moved C3 26.1 mm to (81.3, 17.8)
- moved C2 17.3 mm to (77.5, 22.9)
- moved J1 17.0 mm to (91.4, 26.0)
- moved IC2 16.8 mm to (80.0, 10.2)
- moved D1 16.6 mm to (72.4, 17.1)
- moved U$1 16.6 mm to (83.8, 23.5)
- moved LED1 16.0 mm to (67.9, 13.3)
- moved R2 16.0 mm to (67.9, 19.7)
- moved C1 15.5 mm to (69.2, 24.8)
- moved C4 15.1 mm to (8.89, 25.4), turned to 180 degrees
- moved IC1 9.38 mm to (38.7, 17.8)
- moved U1 8.82 mm to (42.5, 10.2)
Connections:
- net D0/RX renamed N$7
- net D1/TX renamed N$8
- net +5V: now also C1.1, C3.+, RF.2; no longer C1.+, C3.1, JP2.3
- net D10: now also KEYPAD.7; no longer SV1.6
- net D11: now also KEYPAD.8; no longer SV1.7
- net D12: no longer SV1.8
- net D2: no longer JP2.4
- net D3: now also RF.3
- net D4: now also KEYPAD.1
- net D5: now also KEYPAD.2; no longer SV1.1
- net D6: now also KEYPAD.3; no longer SV1.2
- net D7: now also KEYPAD.4; no longer SV1.3
- net D8: now also KEYPAD.5; no longer SV1.4
- net D9: now also KEYPAD.6; no longer SV1.5
- net GND: now also C1.2, C3.-, J1.GND, J1.GNDBREAK, RF.1; no longer C1.-, C3.2, JP2.2
Routing:
- net GND: track 52.7 -> 162.7 mm
- net +5V: track 50.3 -> 129.1 mm
- net N$8: track 0.00 -> 34.6 mm
- net D4: track 0.00 -> 31.5 mm
- net N$7: track 0.00 -> 29.6 mm
- net N$4: track 0.00 -> 28.6 mm
- net D3: track 0.00 -> 23.8 mm
- net D5: track 0.00 -> 16.4 mm
- net D11: track 0.00 -> 15.8 mm
- net D6: track 0.00 -> 13.9 mm
- net D7: track 0.00 -> 11.4 mm
- net D10: track 0.00 -> 10.3 mm
- net D8: track 0.00 -> 8.83 mm
- net D9: track 0.00 -> 7.25 mm
- net EXT_RESET: track 0.00 -> 3.81 mm
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- added copper zone on layer 16, net N$6
- added copper zone on layer 1, net N$9
