File: layout/prototype.sch (EAGLE design)
At the start: 9 parts, among them IC1 ATMEGA328", U1 RESONATOR"

Commit message: Finish controler layout!
Parts:
- added C1: 0.1uF, RBBB:UNPOLARIZED_CAP"
- added C2: 47uF, RBBB:ELECTROLYTIC_CAP2.54MM
- added D1: 1N4004, diode:1N4004
- added IC2: (no value), RBBB:REGULATOR
- added J1: POWER_JACK", RBBB:POWER_JACK"
- added KEYPAD: 1X09_HEADER", RBBB:1X09_HEADER"
- added RF: (no value), RBBB:1X04_HEADER"
- added U$1: 1X02_HEADER, RBBB:1X02_HEADER
- C3: value 0.1uF -> 47uF
Connections:
- net D0/RX renamed N$7
- net D1/TX renamed N$8
- new net N$5: C2.+, D1.C, IC2.IN, J1.PWR, U$1.1
- net +5V: now also C1.1, IC2.OUT, RF.2
- net D10: now also KEYPAD.7
- net D11: now also KEYPAD.8
- net D3: now also RF.3
- net D4: now also KEYPAD.1
- net D5: now also KEYPAD.2
- net D6: now also KEYPAD.3
- net D7: now also KEYPAD.4
- net D8: now also KEYPAD.5
- net D9: now also KEYPAD.6
- net GND: now also C1.2, C2.-, D1.A, IC2.GND, J1.GND, J1.GNDBREAK, RF.1, U$1.2
Other:
- moved on the sheet: C3
