File: Layout_station/untitled.sch (EAGLE design)
At the start: 16 parts, among them IC1 ATMEGA328"

Commit message: "Station" layout completed! Readme updated!
Parts:
- added 12V_INPUT, LIMIT_SW: 1X02_HEADER, RBBB:1X02_HEADER
- added AD_INPUT, EXTERN_PIN: (no value), RBBB:1X04_HEADER"
- added BT, M1, M2: (no value), RBBB:1X06_HEADER"
- added LED1: (no value), RBBB:LED3MM
- added R10: 330, RBBB:RESISTOR1/6WATT
- added R12: 10K, RBBB:RESISTOR1/6WATT
- added S2: MOMENTARY_SWITCH", RBBB:MOMENTARY_SWITCH"
Connections:
- new net EN: BT.6
- new net N$12: IC2.O1, M1.4
- new net N$13: IC2.O2, M1.3
- new net N$14: IC2.O3, M1.2
- new net N$15: IC2.O4, M1.1
- new net N$16: IC2.O5, M2.4
- new net N$17: IC2.O6, M2.3
- new net N$18: IC2.O7, M2.2
- new net N$19: IC2.O8, M2.1
- new net N$20: LED1.A, R10.1
- new net STATE: BT.1
- net +12V: now also 12V_INPUT.2, M1.5, M2.5
- net +5V: now also BT.5, R12.2
- net A0: now also AD_INPUT.1
- net A1: now also AD_INPUT.2
- net A2: now also AD_INPUT.3
- net A3: now also LIMIT_SW.1, R12.1, S2.1
- net A4: now also EXTERN_PIN.1
- net A5: now also EXTERN_PIN.2
- net D13: now also R10.2
- net D2: now also BT.3
- net D3: now also BT.2
- net D4: now also EXTERN_PIN.3
- net GND: now also 12V_INPUT.1, AD_INPUT.4, BT.4, EXTERN_PIN.4, LED1.C, LIMIT_SW.2, S2.2
